Commit message: new

File: install/tb3 gazebo mit sonar/Files mit Sonar/turtlebot3_burger.urdf (robot description, URDF)
Before this commit: robot turtlebot3_burger, 9 links, 8 joints
Links:
- removed link base_sonar_front_left
- removed link base_sonar_front_right
- added link sonar_link, mass 1e-5; collision box size=0.01 0.01 0.01; visual box size=0.01 0.01 0.01
Joints:
- removed joint sonar_front_joint_left
- removed joint sonar_front_joint_right
- added joint sonar_joint: type fixed, parent base_link, child sonar_link, origin xyz=0.04 0.06 0.10 rpy=0 -0.12 0.2, axis 0 1 0
