Commit message: VErsion Vorlesung

File: install/tb3 gazebo mit Range Sensor/Files mit Range Sensor/1x Range Scan worx/turtlebot3_burger.urdf (robot description, URDF)
Before this commit: robot turtlebot3_burger, 8 links, 7 joints
Links:
- link range_scan: geometry collision box size=0.030 0.03 0.02; visual box size=0.030 0.03 0.02
